File: PCB/Acesstra V2/V2.brd (EAGLE design)
At the start: 160 x 100 mm, 15 parts, among them K1 HLS8L-DC5V-S-C, Q1 2N2222

Commit message: Ajustes na PCB
Parts:
- moved S1 72.4 mm to (78.7, 48.3), turned to 180 degrees
- moved K1 66.1 mm to (87.6, 12.7)
- moved D1 63.7 mm to (83.8, 27.9), turned to 180 degrees
- moved ARDUINO_NANO1 51.8 mm to (69.8, 76.2), turned to 270 degrees
- moved R4 50.8 mm to (82.5, 36.8)
- moved R3 47.4 mm to (47.0, 95.2)
- moved Q1 25.0 mm to (59.7, 12.7)
- moved U$1 9.25 mm to (29.2, 73.7)
- moved R5 4.02 mm to (11.4, 40.6)
- moved R1 3.81 mm to (129.5, 31.8)
- moved R2 2.84 mm to (129.5, 47.0)
- turned SG1 to 90 degrees
Routing:
- net N$17: track 425.8 -> 68.8 mm
- net N$12: track 369.7 -> 95.4 mm
- net N$9: track 657.2 -> 393.0 mm
- net N$5: track 347.0 -> 87.4 mm
- net N$10: track 324.0 -> 70.7 mm
- net N$4: track 292.6 -> 82.9 mm
- net N$15: track 202.8 -> 18.9 mm
- net N$1: track 261.7 -> 93.4 mm
- net N$2: track 142.8 -> 13.2 mm
- net N$18: track 135.3 -> 28.3 mm
- net N$19: track 129.5 -> 25.0 mm
- net N$11: track 128.3 -> 35.2 mm
- net N$13: track 5.37 -> 70.4 mm
- net N$16: track 112.6 -> 69.3 mm
- net N$14: track 0.00 -> 30.2 mm
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- added copper zone on layer 16, net GND

Commit message: Ajuste da PCB
Parts:
- moved R3 109.1 mm to (1.27, -3.81)
Connections:
- removed net 5V: U$1.5
- net N$10: now also U$1.5
- net N$15: now also M1.MISO, R3.2; no longer R3.1, U$1.13
- net N$16: now also R3.1, U$1.13; no longer M1.MISO, R3.2
Routing:
- net N$15: track 18.9 -> 0.00 mm
- net N$16: track 69.3 -> 87.8 mm
Changed lines of the file:
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@@
 <attribute name="VALUE" x="127.4064" y="44.6786" size="0.9906" layer="27" ratio="10"/>
-</element>
-<element name="R3" library="rcl" library_urn="urn:adsk.eagle:library:334" package="0204/5" package3d_urn="urn:adsk.eagle:package:23488/1" value="10k" x="46.99" y="95.25" smashed="yes">
-<attribute name="NAME" x="44.9834" y="96.4184" size="0.9906" layer="25" ratio="10"/>
-<attribute name="POPULARITY" value="18" x="129.54" y="-26.67" size="1.778" layer="27" display="off"/>
-<attribute name="SPICEPREFIX" value="R" x="129.54" y="-26.67" size="1.778" layer="27" display="off"/>
-<attribute name="VALUE" x="44.8564" y="92.9386" size="0.9906" layer="27" ratio="10"/>
 </element>
 <element name="R4" library="rcl" library_urn="urn:adsk.eagle:library:334" package="0204/5" package3d_urn="urn:adsk.eagle:package:23488/1" value="10k" x="82.55" y="36.83" smashed="yes">
@@
 <attribute name="NAME" x="29.21" y="57.15" size="1.27" layer="25" rot="R180" align="bottom-center"/>
 <attribute name="VALUE" x="27.94" y="90.17" size="1.27" layer="27" rot="R180" align="top-center"/>
+</element>
+<element name="R3" library="rcl" library_urn="urn:adsk.eagle:library:334" package="0204/5" package3d_urn="urn:adsk.eagle:package:23488/1" value="10k" x="1.27" y="-3.81" smashed="yes">
+<attribute name="NAME" x="-0.7366" y="-2.6416" size="0.9906" layer="25" ratio="10"/>
+<attribute name="POPULARITY" value="18" x="1.27" y="-3.81" size="1.778" layer="27" display="off"/>
+<attribute name="SPICEPREFIX" value="R" x="1.27" y="-3.81" size="1.778" layer="27" display="off"/>
+<attribute name="VALUE" x="-0.8636" y="-6.1214" size="0.9906" layer="27" ratio="10"/>
 </element>
 </elements>
@@
 <signal name="GND.1" class="1">
 <contactref element="U$1" pad="1"/>
-</signal>
-<signal name="5V" class="1">
-<contactref element="U$1" pad="5"/>
 </signal>
 <signal name="N$1">
@@
 <wire x1="57.2897" y1="12.7127" x2="57.15" y2="12.7" width="0.508" layer="16"/>
 <wire x1="75.2856" y1="45.8978" x2="75.4888" y2="45.9994" width="0.508" layer="16"/>
+<contactref element="U$1" pad="5"/>
+<wire x1="62.23" y1="68.58" x2="50.8" y2="69.85" width="0" layer="19" extent="1-1"/>
 </signal>
 <signal name="N$9">
@@
 <wire x1="100.2157" y1="71.1581" x2="100.33" y2="71.12" width="0.508" layer="16"/>
 </signal>
-<signal name="N$15">
-<contactref element="U$1" pad="13"/>
-<contactref element="R3" pad="1"/>
-<wire x1="44.577" y1="84.5312" x2="44.577" y2="95.0976" width="0.508" layer="16"/>
-<wire x1="47.879" y1="81.2292" x2="44.577" y2="84.5312" width="0.508" layer="16"/>
-<wire x1="49.53" y1="81.2292" x2="47.879" y2="81.2292" width="0.508" layer="16"/>
-<wire x1="50.6857" y1="80.0735" x2="49.53" y2="81.2292" width="0.508" layer="16"/>
-<wire x1="44.577" y1="95.0976" x2="44.45" y2="95.25" width="0.508" layer="16"/>
-<wire x1="50.6857" y1="80.0735" x2="50.8" y2="80.01" width="0.508" layer="16"/>
-</signal>
 <signal name="N$16">
-<contactref element="M1" pad="MISO"/>
-<contactref element="R3" pad="2"/>
 <contactref element="ARDUINO_NANO1" pad="30"/>
 <wire x1="64.0588" y1="96.4184" x2="77.4319" y2="96.4184" width="0.508" layer="16"/>
@@
 <wire x1="49.53" y1="95.2627" x2="62.9031" y2="95.2627" width="0.508" layer="16"/>
 <wire x1="77.4319" y1="96.4184" x2="77.47" y2="96.52" width="0.508" layer="16"/>
-<wire x1="49.53" y1="95.2627" x2="49.53" y2="95.25" width="0.508" layer="16"/>
 <wire x1="101.3714" y1="78.7527" x2="100.3808" y2="78.7527" width="0.508" layer="16"/>
 <wire x1="103.6828" y1="81.0641" x2="101.3714" y2="78.7527" width="0.508" layer="16"/>
@@
 <wire x1="94.9325" y1="96.2533" x2="103.6828" y2="87.503" width="0.508" layer="16"/>
 <wire x1="77.597" y1="96.2533" x2="94.9325" y2="96.2533" width="0.508" layer="16"/>
-<wire x1="100.3808" y1="78.7527" x2="100.33" y2="78.74" width="0.508" layer="16"/>
 <wire x1="77.597" y1="96.2533" x2="77.47" y2="96.52" width="0.508" layer="16"/>
+<contactref element="U$1" pad="13"/>
+<wire x1="44.577" y1="84.5312" x2="44.577" y2="95.0976" width="0.508" layer="16"/>
+<wire x1="47.879" y1="81.2292" x2="44.577" y2="84.5312" width="0.508" layer="16"/>
+<wire x1="49.53" y1="81.2292" x2="47.879" y2="81.2292" width="0.508" layer="16"/>
+<wire x1="50.6857" y1="80.0735" x2="49.53" y2="81.2292" width="0.508" layer="16"/>
+<wire x1="50.6857" y1="80.0735" x2="50.8" y2="80.01" width="0.508" layer="16"/>
+<contactref element="R3" pad="1"/>
+<wire x1="44.577" y1="95.0976" x2="49.53" y2="95.2627" width="0" layer="19" extent="16-16"/>
+<wire x1="-1.27" y1="-3.81" x2="50.8" y2="80.01" width="0" layer="19" extent="1-1"/>
 </signal>
 <signal name="N$17">
-<contactref element="M1" pad="MOSI"/>
 <contactref element="U$1" pad="9"/>
 <contactref element="ARDUINO_NANO1" pad="29"/>
@@
 <wire x1="100.3808" y1="81.3943" x2="102.362" y2="83.3755" width="0.508" layer="16"/>
 <wire x1="77.597" y1="93.9419" x2="77.47" y2="93.98" width="0.508" layer="16"/>
-<wire x1="100.3808" y1="81.3943" x2="100.33" y2="81.28" width="0.508" layer="16"/>
 <wire x1="51.8414" y1="74.9554" x2="50.8508" y2="74.9554" width="0.508" layer="16"/>
 <wire x1="62.0776" y1="85.1916" x2="51.8414" y2="74.9554" width="0.508" layer="16"/>
@@
 <wire x1="50.8508" y1="74.9554" x2="50.8" y2="74.93" width="0.508" layer="16"/>
 <wire x1="77.2668" y1="93.9419" x2="77.47" y2="93.98" width="0.508" layer="16"/>
+<contactref element="M1" pad="MOSI"/>
+<wire x1="100.3808" y1="81.3943" x2="100.33" y2="81.28" width="0" layer="19" extent="16-16"/>
 </signal>
 <signal name="N$18">
@@
 <wire x1="62.0776" y1="96.5835" x2="62.23" y2="96.52" width="0.508" layer="16"/>
 </signal>
+<signal name="N$15">
+<contactref element="M1" pad="MISO"/>
+<contactref element="R3" pad="2"/>
+<wire x1="3.81" y1="-3.81" x2="100.33" y2="78.74" width="0" layer="19" extent="1-1"/>
+</signal>
 </signals>
